Commit message: Fixed steer left drift (use fixed joints), and add gitignore

File: src/rb2301_gz/urdf/nanocar_description.urdf (robot description, URDF)
Before this commit: robot NanoCar, 9 links, 8 joints
Joints:
- joint back_left_wheel_joint: type continuous -> fixed
- joint back_right_wheel_joint: type continuous -> fixed
- joint front_left_wheel_joint: type continuous -> fixed
- joint front_right_wheel_joint: type continuous -> fixed
